File: hardware/hardware.kicad_sch (KiCad schematic)
At the start: 40 parts, among them J1 Conn_01x06, J2 USB_C_Receptacle_USB2.0_14P, J3 Conn_01x04_Pin, Q1 BSS138, Q2 BSS138, U1 CH340C, U2 ESP32-WROOM-32, U3 AMS1117-3.3, U4 DRV8825PWPR

Commit message: finish pcb wiring
Parts:
- added J4: Conn_01x02_Pin, Connector_JST:JST_XH_B2B-XH-A_1x02_P2.50mm_Vertical, symbol Connector:Conn_01x02_Pin
- J3: footprint TerminalBlock_Phoenix:TerminalBlock_Phoenix_MPT-0,5-4-2.54_1x04_P2.54mm_Horizontal -> Connector_JST:JST_XH_B4B-XH-A_1x04_P2.50mm_Vertical
Connections:
- net +BATT is gone; now on net +5V: C7.1, C9.1, R7.2, U4.11 (VMB), U4.4 (VMA)
- net +3.3V: now also JP1.3 (B), JP2.3 (B), JP3.3 (B), R9.2
- net +5V: now also J4.2 (Pin_2)
- net DIR: now also U2.29 (IO5)
- net GND: now also J4.1 (Pin_1)
- net STEP: now also U2.26 (IO4)
- net VBUS: no longer JP1.3 (B), JP2.3 (B), JP3.3 (B), R9.2
- net at J3.1 (Pin_1): now also U4.7 (AOUT2); no longer U4.8 (BOUT2)
- net at J3.2 (Pin_2): now also U4.5 (AOUT1); no longer U4.10 (BOUT1)
- net at J3.3 (Pin_3): now also U4.10 (BOUT1); no longer U4.5 (AOUT1)
- net at J3.4 (Pin_4): now also U4.8 (BOUT2); no longer U4.7 (AOUT2)
Other:
- moved on the sheet: J3
